Commit message: feat: Refactor mobile robot simulation workspace for clarity and usability.
- Replace the cave simulation with an example indoor test scene in `robot_bringup`.
- Update README to reflect new launch commands and scene descriptions.
- Introduce detailed documentation for each package, including `robot_description`, `robot_control`, and `robot_gazebo`.
- Add support for custom mesh scene imports and improve launch file parameters.
- Remove outdated cave world files and streamline the overall structure.

This update enhances the user experience and provides clearer guidance for simulation setup.

File: src/robot_control/urdf/robot.ros2_control.xacro (robot description, xacro)
@@ -1,5 +1,5 @@
 <?xml version="1.0"?>
 <robot xmlns:xacro="http://www.ros.org/wiki/xacro">
-  <xacro:macro name="cave_robot_ros2_control">
+  <xacro:macro name="robot_ros2_control">
     <ros2_control name="GazeboSimSystem" type="system">
       <hardware>

File: src/robot_description/urdf/chassis.xacro (robot description, xacro)
@@ -8,4 +8,5 @@
   <xacro:property name="chassis_width" value="0.4"/>
   <xacro:property name="chassis_height" value="0.3"/>
+  <xacro:property name="ground_clearance" value="0.08"/>
   <xacro:property name="track_width" value="0.5"/>
   <xacro:property name="wheelbase" value="0.4"/>
@@ -37,28 +38,4 @@
     </inertial>
   </link>
-  <link name="lidar_mast_link">
-    <visual>
-      <geometry>
-        <cylinder radius="0.03" length="0.35"/>
-      </geometry>
-      <material name="black">
-        <color rgba="0.1 0.1 0.1 1.0"/>
-      </material>
-    </visual>
-    <collision>
-      <geometry>
-        <cylinder radius="0.03" length="0.35"/>
-      </geometry>
-    </collision>
-    <inertial>
-      <mass value="0.5"/>
-      <inertia ixx="0.01" ixy="0" ixz="0" iyy="0.01" iyz="0" izz="0.01"/>
-    </inertial>
-  </link>
-  <joint name="lidar_mast_joint" type="fixed">
-    <parent link="base_link"/>
-    <child link="lidar_mast_link"/>
-    <origin xyz="0 0 ${chassis_height * 0.5 + 0.175}" rpy="0 0 0"/>
-  </joint>
   <xacro:macro name="wheel" params="prefix x y mimic_joint:='none'">
     <link name="${prefix}_wheel_link">
@@ -83,5 +60,5 @@
       <parent link="base_link"/>
       <child link="${prefix}_wheel_link"/>
-      <origin xyz="${x} ${y} ${-(chassis_height * 0.5 - wheel_radius)}" rpy="0 0 0"/>
+      <origin xyz="${x} ${y} ${-(chassis_height * 0.5 - wheel_radius + ground_clearance)}" rpy="0 0 0"/>
       <axis xyz="0 1 0"/>
       <xacro:unless value="${mimic_joint == 'none'}">
@@ -90,15 +67,10 @@
     </joint>
   </xacro:macro>
-  <gazebo reference="lidar_mast_link">
-    <material>
-      <ambient>0.1 0.1 0.1 1</ambient>
-      <diffuse>0.1 0.1 0.1 1</diffuse>
-    </material>
-  </gazebo>
-  <xacro:wheel prefix="left_front" x="${wheelbase * 0.5}" y="${-track_width * 0.5}"/>
-  <xacro:wheel prefix="right_front" x="${wheelbase * 0.5}" y="${track_width * 0.5}"/>
-  <xacro:wheel prefix="left_rear" x="${-wheelbase * 0.5}" y="${-track_width * 0.5}"
+  <!-- REP-103: +Y is left, -Y is right -->
+  <xacro:wheel prefix="left_front" x="${wheelbase * 0.5}" y="${track_width * 0.5}"/>
+  <xacro:wheel prefix="right_front" x="${wheelbase * 0.5}" y="${-track_width * 0.5}"/>
+  <xacro:wheel prefix="left_rear" x="${-wheelbase * 0.5}" y="${track_width * 0.5}"
                mimic_joint="left_front_wheel_joint"/>
-  <xacro:wheel prefix="right_rear" x="${-wheelbase * 0.5}" y="${track_width * 0.5}"
+  <xacro:wheel prefix="right_rear" x="${-wheelbase * 0.5}" y="${-track_width * 0.5}"
                mimic_joint="right_front_wheel_joint"/>
   <gazebo reference="base_link">

File: src/robot_description/urdf/lidar.xacro (robot description, xacro)
@@ -4,6 +4,16 @@
     <visual>
       <geometry>
+        <box size="0.08 0.08 0.02"/>
+      </geometry>
+      <origin xyz="0 0 0.045" rpy="0 0 0"/>
+      <material name="lidar_mount_gray">
+        <color rgba="0.2 0.2 0.2 1.0"/>
+      </material>
+    </visual>
+    <visual>
+      <geometry>
         <cylinder radius="0.055" length="0.07"/>
       </geometry>
+      <origin xyz="0 0 0.08" rpy="0 0 0"/>
       <material name="lidar_gray">
         <color rgba="0.3 0.3 0.3 1.0"/>
@@ -14,14 +24,16 @@
         <cylinder radius="0.055" length="0.07"/>
       </geometry>
+      <origin xyz="0 0 0.08" rpy="0 0 0"/>
     </collision>
     <inertial>
       <mass value="0.3"/>
+      <origin xyz="0 0 0.04" rpy="0 0 0"/>
       <inertia ixx="0.001" ixy="0" ixz="0" iyy="0.001" iyz="0" izz="0.001"/>
     </inertial>
   </link>
   <joint name="lidar_joint" type="fixed">
-    <parent link="lidar_mast_link"/>
+    <parent link="base_link"/>
     <child link="lidar_link"/>
-    <origin xyz="0 0 0.21" rpy="0 0 0"/>
+    <origin xyz="0 0 ${chassis_height * 0.5 + 0.04}" rpy="0 0 0"/>
   </joint>
   <gazebo reference="lidar_link">
@@ -36,4 +48,5 @@
       <topic>/lidar/scan</topic>
       <gz_frame_id>lidar_link</gz_frame_id>
+      <pose>0 0 0.08 0 0 0</pose>
       <ray>
         <scan>
@@ -53,5 +66,5 @@
         <range>
           <min>0.1</min>
-          <max>100.0</max>
+          <max>50.0</max>
           <resolution>0.01</resolution>
         </range>

File: src/robot_description/urdf/robot.urdf.xacro (robot description, xacro)
@@ -1,4 +1,4 @@
 <?xml version="1.0"?>
-<robot xmlns:xacro="http://www.ros.org/wiki/xacro" name="cave_robot">
+<robot xmlns:xacro="http://www.ros.org/wiki/xacro" name="robot">
   <xacro:arg name="wheel_joint_type" default="fixed"/>
   <xacro:arg name="use_diff_drive" default="false"/>
@@ -15,5 +15,5 @@
   <xacro:if value="$(arg use_ros2_control)">
     <xacro:include filename="$(find robot_control)/urdf/robot.ros2_control.xacro"/>
-    <xacro:cave_robot_ros2_control/>
+    <xacro:robot_ros2_control/>
   </xacro:if>
 </robot>
