Commit message: refactor: Remove robot_control package and update documentation
- Deleted the `robot_control` package, including its configuration files and dependencies.
- Updated README and documentation to reflect the removal of `robot_control` and clarified the use of the Gazebo DiffDrive plugin.
- Adjusted launch files and package dependencies accordingly to streamline the simulation setup.
- Enhanced clarity in the documentation regarding the simulation environment and its components.

File: src/robot_description/urdf/robot.urdf.xacro (robot description, xacro)
@@ -3,8 +3,6 @@
   <xacro:arg name="wheel_joint_type" default="fixed"/>
   <xacro:arg name="use_diff_drive" default="false"/>
-  <xacro:arg name="use_ros2_control" default="false"/>
   <xacro:property name="wheel_joint_type" value="$(arg wheel_joint_type)"/>
   <xacro:property name="use_diff_drive" value="$(arg use_diff_drive)"/>
-  <xacro:property name="use_ros2_control" value="$(arg use_ros2_control)"/>
   <xacro:property name="chassis_length" value="0.6"/>
   <xacro:include filename="chassis.xacro"/>
@@ -13,7 +11,3 @@
   <xacro:include filename="camera.xacro"/>
   <xacro:include filename="gazebo_plugins.xacro"/>
-  <xacro:if value="$(arg use_ros2_control)">
-    <xacro:include filename="$(find robot_control)/urdf/robot.ros2_control.xacro"/>
-    <xacro:robot_ros2_control/>
-  </xacro:if>
 </robot>
