Commit message: feat: extract drive plugins and fix mecanum odometry bridge
Split drivetrain plugin definitions into quadrover_control and switch launch flow to drive_mode-based control only. Add mecanum-specific OdometryWithCovariance bridge remapping so /odom/wheel publishes consistently across drive modes.

Co-authored-by: Cursor <cursoragent@cursor.com>

File: src/quadrover_description/urdf/camera.xacro (robot description, xacro)
@@ -26,8 +26,4 @@
   </joint>
   <gazebo reference="camera_link">
-    <material>
-      <ambient>0.1 0.1 0.8 1</ambient>
-      <diffuse>0.1 0.1 0.8 1</diffuse>
-    </material>
     <sensor name="rgb_camera" type="camera">
       <always_on>true</always_on>

File: src/quadrover_description/urdf/chassis.xacro (robot description, xacro)
@@ -74,18 +74,8 @@
   <xacro:wheel prefix="right_rear" x="${-wheelbase * 0.5}" y="${-track_width * 0.5}"
                mimic_joint="right_front_wheel_joint"/>
-  <gazebo reference="base_link">
-    <material>
-      <ambient>0.8 0.1 0.1 1</ambient>
-      <diffuse>0.8 0.1 0.1 1</diffuse>
-    </material>
-  </gazebo>
   <xacro:macro name="wheel_gazebo" params="prefix">
     <gazebo reference="${prefix}_wheel_link">
       <mu1>1.0</mu1>
       <mu2>1.0</mu2>
-      <material>
-        <ambient>0.05 0.05 0.05 1</ambient>
-        <diffuse>0.05 0.05 0.05 1</diffuse>
-      </material>
     </gazebo>
   </xacro:macro>

File: src/quadrover_description/urdf/gazebo_plugins.xacro (robot description, xacro)
@@ -1,36 +1,4 @@
 <?xml version="1.0"?>
 <robot xmlns:xacro="http://www.ros.org/wiki/xacro">
-  <xacro:if value="$(arg use_diff_drive)">
-    <gazebo>
-      <plugin filename="gz-sim-diff-drive-system" name="gz::sim::systems::DiffDrive">
-        <left_joint>left_front_wheel_joint</left_joint>
-        <left_joint>left_rear_wheel_joint</left_joint>
-        <right_joint>right_front_wheel_joint</right_joint>
-        <right_joint>right_rear_wheel_joint</right_joint>
-        <wheel_separation>0.5</wheel_separation>
-        <wheel_radius>0.15</wheel_radius>
-        <odom_publish_frequency>30</odom_publish_frequency>
-        <topic>/cmd_vel</topic>
-        <odom_topic>/odom/wheel</odom_topic>
-        <tf_topic>/odom/wheel/tf_internal</tf_topic>
-        <frame_id>odom</frame_id>
-        <child_frame_id>base_link</child_frame_id>
-        <max_linear_acceleration>1.0</max_linear_acceleration>
-        <min_linear_acceleration>-1.0</min_linear_acceleration>
-        <max_angular_acceleration>2.0</max_angular_acceleration>
-        <min_angular_acceleration>-2.0</min_angular_acceleration>
-        <max_linear_velocity>1.0</max_linear_velocity>
-        <min_linear_velocity>-1.0</min_linear_velocity>
-        <max_angular_velocity>1.5</max_angular_velocity>
-        <min_angular_velocity>-1.5</min_angular_velocity>
-      </plugin>
-    </gazebo>
-    <gazebo>
-      <plugin filename="gz-sim-joint-state-publisher-system"
-              name="gz::sim::systems::JointStatePublisher">
-        <topic>/joint_states</topic>
-      </plugin>
-    </gazebo>
-  </xacro:if>
   <gazebo>
     <plugin filename="ignition-gazebo-odometry-publisher-system"

File: src/quadrover_description/urdf/lidar.xacro (robot description, xacro)
@@ -38,8 +38,4 @@
   </joint>
   <gazebo reference="lidar_link">
-    <material>
-      <ambient>0.3 0.3 0.3 1</ambient>
-      <diffuse>0.3 0.3 0.3 1</diffuse>
-    </material>
     <sensor name="lidar" type="gpu_lidar">
       <always_on>true</always_on>

File: src/quadrover_description/urdf/quadrover.urdf.xacro (robot description, xacro)
@@ -1,8 +1,7 @@
 <?xml version="1.0"?>
 <robot xmlns:xacro="http://www.ros.org/wiki/xacro" name="quadrover">
-  <xacro:arg name="wheel_joint_type" default="fixed"/>
-  <xacro:arg name="use_diff_drive" default="false"/>
-  <xacro:property name="wheel_joint_type" value="$(arg wheel_joint_type)"/>
-  <xacro:property name="use_diff_drive" value="$(arg use_diff_drive)"/>
+  <xacro:arg name="drive_mode" default="diff_drive"/>
+  <xacro:property name="wheel_joint_type" value="continuous"/>
+  <xacro:property name="drive_mode" value="$(arg drive_mode)"/>
   <xacro:property name="chassis_length" value="0.6"/>
   <xacro:include filename="chassis.xacro"/>
@@ -10,4 +9,5 @@
   <xacro:include filename="lidar.xacro"/>
   <xacro:include filename="camera.xacro"/>
+  <xacro:include filename="$(find quadrover_control)/urdf/drive_plugins.xacro"/>
   <xacro:include filename="gazebo_plugins.xacro"/>
 </robot>
