Commit message: refactor: simplify to diff-drive only and remove odom TF scripts
Drop mecanum drive, wheel odom normalizer, and launch TF options; bridge
/odom/wheel directly from Gazebo DiffDrive and align all docs with the
simplified runtime.

Co-authored-by: Cursor <cursoragent@cursor.com>

File: src/quadrover_control/urdf/drive_plugins.xacro (robot description, xacro)
@@ -1,49 +1,28 @@
 <?xml version="1.0"?>
 <robot xmlns:xacro="http://www.ros.org/wiki/xacro">
-  <xacro:if value="${drive_mode == 'diff_drive'}">
-    <gazebo>
-      <plugin filename="gz-sim-diff-drive-system" name="gz::sim::systems::DiffDrive">
-        <left_joint>left_front_wheel_joint</left_joint>
-        <left_joint>left_rear_wheel_joint</left_joint>
-        <right_joint>right_front_wheel_joint</right_joint>
-        <right_joint>right_rear_wheel_joint</right_joint>
-        <wheel_separation>0.5</wheel_separation>
-        <wheel_radius>0.15</wheel_radius>
-        <odom_publish_frequency>30</odom_publish_frequency>
-        <topic>/cmd_vel</topic>
-        <odom_topic>/odom/wheel</odom_topic>
-        <tf_topic>/odom/wheel/tf_internal</tf_topic>
-        <frame_id>odom</frame_id>
-        <child_frame_id>base_link</child_frame_id>
-        <max_linear_acceleration>1.0</max_linear_acceleration>
-        <min_linear_acceleration>-1.0</min_linear_acceleration>
-        <max_angular_acceleration>2.0</max_angular_acceleration>
-        <min_angular_acceleration>-2.0</min_angular_acceleration>
-        <max_linear_velocity>1.0</max_linear_velocity>
-        <min_linear_velocity>-1.0</min_linear_velocity>
-        <max_angular_velocity>1.5</max_angular_velocity>
-        <min_angular_velocity>-1.5</min_angular_velocity>
-      </plugin>
-    </gazebo>
-  </xacro:if>
-  <xacro:if value="${drive_mode == 'mecanum_drive'}">
-    <gazebo>
-      <plugin filename="ignition-gazebo-mecanum-drive-system" name="ignition::gazebo::systems::MecanumDrive">
-        <front_left_joint>left_front_wheel_joint</front_left_joint>
-        <back_left_joint>left_rear_wheel_joint</back_left_joint>
-        <front_right_joint>right_front_wheel_joint</front_right_joint>
-        <back_right_joint>right_rear_wheel_joint</back_right_joint>
-        <wheel_separation>0.5</wheel_separation>
-        <wheel_base>0.4</wheel_base>
-        <wheel_radius>0.15</wheel_radius>
-        <odom_publish_frequency>30</odom_publish_frequency>
-        <topic>/cmd_vel</topic>
-        <odom_topic>/odom/wheel</odom_topic>
-        <tf_topic>/odom/wheel/tf_internal</tf_topic>
-        <frame_id>odom</frame_id>
-        <child_frame_id>base_link</child_frame_id>
-      </plugin>
-    </gazebo>
-  </xacro:if>
+  <gazebo>
+    <plugin filename="gz-sim-diff-drive-system" name="gz::sim::systems::DiffDrive">
+      <left_joint>left_front_wheel_joint</left_joint>
+      <left_joint>left_rear_wheel_joint</left_joint>
+      <right_joint>right_front_wheel_joint</right_joint>
+      <right_joint>right_rear_wheel_joint</right_joint>
+      <wheel_separation>0.5</wheel_separation>
+      <wheel_radius>0.15</wheel_radius>
+      <odom_publish_frequency>30</odom_publish_frequency>
+      <topic>/cmd_vel</topic>
+      <odom_topic>/odom/wheel</odom_topic>
+      <tf_topic>/odom/wheel/tf_internal</tf_topic>
+      <frame_id>odom</frame_id>
+      <child_frame_id>base_link</child_frame_id>
+      <max_linear_acceleration>1.0</max_linear_acceleration>
+      <min_linear_acceleration>-1.0</min_linear_acceleration>
+      <max_angular_acceleration>2.0</max_angular_acceleration>
+      <min_angular_acceleration>-2.0</min_angular_acceleration>
+      <max_linear_velocity>1.0</max_linear_velocity>
+      <min_linear_velocity>-1.0</min_linear_velocity>
+      <max_angular_velocity>1.5</max_angular_velocity>
+      <min_angular_velocity>-1.5</min_angular_velocity>
+    </plugin>
+  </gazebo>
   <gazebo>
     <plugin filename="gz-sim-joint-state-publisher-system"

File: src/quadrover_description/urdf/quadrover.urdf.xacro (robot description, xacro)
@@ -1,7 +1,5 @@
 <?xml version="1.0"?>
 <robot xmlns:xacro="http://www.ros.org/wiki/xacro" name="quadrover">
-  <xacro:arg name="drive_mode" default="diff_drive"/>
   <xacro:property name="wheel_joint_type" value="continuous"/>
-  <xacro:property name="drive_mode" value="$(arg drive_mode)"/>
   <xacro:property name="chassis_length" value="0.6"/>
   <xacro:include filename="chassis.xacro"/>
